File: oya38split.kicad_pcb (KiCad board)
At the start: 2 copper layers, 89 parts, among them U1 ProMicro

Commit message: changed layout idea
Parts:
- MX1, MX10, MX11, MX12, MX13, MX14, MX15, MX16, MX17, MX18, MX19, MX2, MX20, MX21, MX22, MX23, MX24, MX25, MX26, MX27, MX28, MX29, MX3, MX30, MX31, MX32, MX33, MX34, MX35, MX36, MX37, MX38, MX39, MX4, MX40, MX41, MX42, MX43, MX44, MX45, MX5, MX6, MX7, MX8, MX9, U1: moved to F.Cu
- moved D38 338.7 mm to (-78.6, 59.8), turned to 0 degrees
- moved D30 329.1 mm to (-72.0, 65.1), turned to 0 degrees
- moved D20 314.9 mm to (-58.9, 62.4), turned to 0 degrees
- moved D43 311.8 mm to (-65.5, 51.8), turned to 0 degrees
- moved D29 303.5 mm to (-65.5, 59.8), turned to 0 degrees
- moved D37 302.8 mm to (-78.6, 62.4), turned to 0 degrees
- moved D42 301.0 mm to (-78.6, 54.5), turned to 0 degrees
- moved D19 300.1 mm to (-65.5, 65.1), turned to 0 degrees
- moved D10 294.9 mm to (-39.3, 55.9), turned to 0 degrees
- moved D36 293.8 mm to (-72.0, 59.8), turned to 0 degrees
- moved U1 280.7 mm to (-142.6, 15.8), turned to 0 degrees
- moved D28 278.9 mm to (-58.9, 54.5), turned to 0 degrees
- moved D18 273.0 mm to (-58.9, 65.1), turned to 0 degrees
- moved D41 271.1 mm to (-72.0, 54.5), turned to 0 degrees
- moved D9 265.7 mm to (-32.7, 55.9), turned to 0 degrees
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Routing:
- net row3: track 199.2 -> 0.00 mm
- net row1: track 198.7 -> 0.00 mm
- net row2: track 198.4 -> 0.00 mm
- net row4: track 198.3 -> 0.00 mm
- net col9: track 188.8 -> 0.00 mm
- net col8: track 150.5 -> 0.00 mm
- net col7: track 150.1 -> 0.00 mm
- net col0: track 144.0 -> 0.00 mm
- net col6: track 133.6 -> 0.00 mm
- net col5: track 125.8 -> 0.00 mm
- net col3: track 112.0 -> 0.00 mm
- net row0: track 110.1 -> 0.00 mm
- net col2: track 107.7 -> 0.00 mm
- net col1: track 106.1 -> 0.00 mm
- net col4: track 102.8 -> 0.00 mm
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
Commit message: fixed layout
Parts:
- MX10, MX16, MX17, MX18, MX19, MX20, MX26, MX27, MX28, MX29, MX30, MX35, MX36, MX37, MX38, MX39, MX40, MX41, MX42, MX43, MX45, MX6, MX7, MX8, MX9: moved to B.Cu
- moved MX10 171.4 mm to (57.1, 57.1), turned to 180 degrees
- moved MX20 171.4 mm to (57.1, 76.2), turned to 180 degrees
- moved MX30 171.4 mm to (57.1, 95.2), turned to 180 degrees
- moved MX38 171.4 mm to (57.1, 114.3), turned to 180 degrees
- moved MX43 152.4 mm to (66.7, 38.1), turned to 180 degrees
- moved MX29 132.4 mm to (77.2, 95.9), turned to 176 degrees
- moved MX19 131.1 mm to (78.5, 76.9), turned to 176 degrees
- moved MX9 129.7 mm to (79.8, 57.9), turned to 176 degrees
- moved MX42 109.4 mm to (90.7, 39.6), turned to 176 degrees
- moved MX37 96.2 mm to (94.4, 116.8), turned to 172 degrees
- moved MX28 93.5 mm to (97.0, 98.0), turned to 172 degrees
- moved MX18 90.9 mm to (99.7, 79.1), turned to 172 degrees
- moved MX8 88.2 mm to (102.3, 60.2), turned to 172 degrees
- moved MX41 66.7 mm to (114.4, 42.7), turned to 172 degrees
- moved MX36 58.4 mm to (113.2, 119.5), turned to 172 degrees
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
Commit message: fixed layout
Parts:
- moved D1 128.1 mm to (-192.9, 123.0)
- moved D10 128.1 mm to (-153.6, 113.8)
- moved D11 128.1 mm to (-147.0, 111.2)
- moved D12 128.1 mm to (-166.7, 115.1)
- moved D15 128.1 mm to (-160.1, 112.4)
- moved D16 128.1 mm to (-166.7, 120.4)
- moved D17 128.1 mm to (-166.7, 117.7)
- moved D19 128.1 mm to (-179.8, 123.0)
- moved D2 128.1 mm to (-160.1, 115.1)
- moved D21 128.1 mm to (-179.8, 120.4)
- moved D23 128.1 mm to (-153.6, 111.2)
- moved D24 128.1 mm to (-186.3, 109.8)
- moved D25 128.1 mm to (-166.7, 112.4)
- moved D26 128.1 mm to (-160.1, 109.8)
- moved D27 128.1 mm to (-166.7, 109.8)
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Other:
- board outline added: 95.2 x 76.2 mm

Commit message: fixed layout
Parts:
- MX10, MX16, MX17, MX18, MX19, MX20, MX26, MX27, MX28, MX29, MX30, MX35, MX36, MX37, MX38, MX39, MX40, MX41, MX42, MX43, MX45, MX6, MX7, MX8, MX9: moved to F.Cu
- moved MX10 208.0 mm to (265.1, 57.1), turned to 0 degrees
- moved MX20 208.0 mm to (265.1, 76.2), turned to 0 degrees
- moved MX30 208.0 mm to (265.1, 95.2), turned to 0 degrees
- moved MX38 208.0 mm to (265.1, 114.3), turned to 0 degrees
- moved MX43 188.9 mm to (255.6, 38.1), turned to 0 degrees
- moved MX29 167.8 mm to (245.0, 96.0), turned to 4 degrees
- moved MX19 165.1 mm to (243.7, 77.0), turned to 4 degrees
- moved MX9 162.4 mm to (242.4, 58.0), turned to 4 degrees
- moved MX42 139.7 mm to (231.0, 39.7), turned to 4 degrees
- moved MX37 133.0 mm to (227.6, 116.9), turned to 8 degrees
- moved MX28 127.7 mm to (225.0, 98.1), turned to 8 degrees
- moved MX18 122.4 mm to (222.3, 79.2), turned to 8 degrees
- moved MX8 117.1 mm to (219.7, 60.3), turned to 8 degrees
- moved MX36 95.3 mm to (208.8, 119.6), turned to 8 degrees
- moved MX41 91.8 mm to (207.0, 42.9), turned to 8 degrees
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
Commit message: fixed layout
Parts:
- MX1, MX10, MX11, MX12, MX13, MX14, MX15, MX16, MX17, MX18, MX19, MX2, MX20, MX21, MX22, MX23, MX24, MX25, MX26, MX27, MX28, MX29, MX3, MX30, MX31, MX32, MX33, MX34, MX35, MX36, MX37, MX38, MX39, MX4, MX40, MX41, MX42, MX43, MX44, MX45, MX5, MX6, MX7, MX8, MX9: moved to B.Cu
- moved D1 323.6 mm to (112.7, 16.7)
- moved D10 323.6 mm to (152.0, 7.44)
- moved D11 323.6 mm to (158.6, 4.79)
- moved D12 323.6 mm to (138.9, 8.72)
- moved D13 323.6 mm to (132.4, 8.72)
- moved D14 323.6 mm to (153.1, 2.14)
- moved D15 323.6 mm to (145.5, 6.07)
- moved D16 323.6 mm to (138.9, 14.0)
- moved D17 323.6 mm to (138.9, 11.4)
- moved D18 323.6 mm to (132.4, 16.7)
- moved D19 323.6 mm to (125.8, 16.7)
- moved D2 323.6 mm to (145.5, 8.72)
- moved D20 323.6 mm to (132.4, 14.0)
- moved D21 323.6 mm to (125.8, 14.0)
- moved D22 323.6 mm to (132.4, 11.4)
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Other:
- board size 95.2 x 76.2 mm -> 217.5 x 106.4 mm

Commit message: fixed layout
Parts:
- moved MX39 14.1 mm to (159.7, 47.9), turned to 188 degrees
- moved MX40 12.6 mm to (178.6, 45.2), turned to 188 degrees
- moved MX6 11.5 mm to (171.6, 65.6), turned to 188 degrees
- moved MX41 11.4 mm to (197.5, 42.6), turned to 188 degrees
- moved MX5 11.0 mm to (140.3, 65.6), turned to 172 degrees
- moved MX7 9.86 mm to (190.5, 63.0), turned to 188 degrees
- moved MX16 9.75 mm to (174.3, 84.5), turned to 188 degrees
- moved MX15 9.35 mm to (137.7, 84.5), turned to 172 degrees
- moved MX4 9.23 mm to (121.5, 63.0), turned to 172 degrees
- moved MX8 8.73 mm to (209.4, 60.3), turned to 188 degrees
- moved MX26 8.48 mm to (176.9, 103.4), turned to 188 degrees
- moved MX25 8.28 mm to (135.0, 103.4), turned to 172 degrees
- moved MX3 8.00 mm to (102.6, 60.3), turned to 172 degrees
- moved MX34 7.99 mm to (132.4, 122.2), turned to 172 degrees
- moved MX35 7.93 mm to (179.6, 122.2), turned to 188 degrees
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Other:
- board size 217.5 x 106.4 mm -> 216.7 x 106.4 mm

Commit message: fixed edgecut
Other:
- board size 216.7 x 106.4 mm -> 216.7 x 104.8 mm
Changed lines of the file:
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@@
   (general
     (thickness 1.6)
-    (drawings 10)
+    (drawings 14)
     (tracks 0)
     (zones 0)
@@
     )
   )
-  (gr_line (start 155.575 134.9375) (end 50.00625 123.825) (layer Edge.Cuts) (width 0.05))
-  (gr_line (start 156.36875 134.9375) (end 155.575 134.9375) (layer Edge.Cuts) (width 0.05))
-  (gr_line (start 261.9375 123.825) (end 156.36875 134.9375) (layer Edge.Cuts) (width 0.05))
+  (gr_line (start 140.49375 133.35) (end 171.45 133.35) (layer Edge.Cuts) (width 0.05))
+  (gr_line (start 83.34375 125.4125) (end 140.49375 133.35) (layer Edge.Cuts) (width 0.05))
+  (gr_line (start 66.675 123.825) (end 83.34375 125.4125) (layer Edge.Cuts) (width 0.05))
+  (gr_line (start 50.00625 123.825) (end 66.675 123.825) (layer Edge.Cuts) (width 0.05))
+  (gr_line (start 228.6 125.4125) (end 171.45 133.35) (layer Edge.Cuts) (width 0.05))
+  (gr_line (start 245.26875 123.825) (end 228.6 125.4125) (layer Edge.Cuts) (width 0.05))
+  (gr_line (start 261.9375 123.825) (end 245.26875 123.825) (layer Edge.Cuts) (width 0.05))
   (gr_line (start 50.00625 28.575) (end 261.9375 28.575) (layer Edge.Cuts) (width 0.05))
   (gr_line (start 264.31875 30.95625) (end 264.31875 121.44375) (layer Edge.Cuts) (width 0.05))

Commit message: arranged diodes
Parts:
- U1: moved to B.Cu
- moved U1 138.8 mm to (67.5, 38.1)
- moved D3 74.6 mm to (78.6, 2.38), turned to 90 degrees
- moved D42 71.5 mm to (171.4, 2.38), turned to 90 degrees
- moved D43 70.9 mm to (173.8, 2.38), turned to 90 degrees
- moved D7 70.9 mm to (88.1, 2.38), turned to 90 degrees
- moved D2 69.6 mm to (76.2, 2.38), turned to 90 degrees
- moved D5 69.4 mm to (83.3, 2.38), turned to 90 degrees
- moved D40 66.7 mm to (166.7, 2.38), turned to 90 degrees
- moved D9 65.9 mm to (92.9, 2.38), turned to 90 degrees
- moved D4 65.8 mm to (81.0, 2.38), turned to 90 degrees
- moved D41 62.8 mm to (169.1, 2.38), turned to 90 degrees
- moved D8 62.0 mm to (90.5, 2.38), turned to 90 degrees
- moved D38 62.0 mm to (161.9, 2.38), turned to 90 degrees
- moved D11 61.0 mm to (97.6, 2.38), turned to 90 degrees
- moved D6 60.6 mm to (85.7, 2.38), turned to 90 degrees
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