File: oya38split.sch (KiCad schematic (older format))
At the start: 89 parts, among them U1 ProMicro

Commit message: added traces and fixed diode
Connections:
- net at D34.2 (A), MX34.2 (ROW): now also MX44.2 (ROW)
- net at D35.2 (A), MX35.2 (ROW): now also MX45.2 (ROW)
Changed lines of the file:
@@
-$EndComp
-$Comp
-L MX_Alps_Hybrid:MX-NoLED MX45
-U 1 1 6141B38D
-P 8050 5350
-F 0 "MX45" H 8083 5573 60  0000 C CNN
-F 1 "MX-NoLED" H 8083 5499 20  0000 C CNN
-F 2 "MX_Only:MXOnly-2U-ReversedStabilizers-NoLED" H 7425 5325 60  0001 C CNN
-F 3 "" H 7425 5325 60  0001 C CNN
-	1    8050 5350
-	1    0    0    -1
 $EndComp
 $Comp
@@
 Text GLabel 2300 3700 0    50   Input ~ 0
 col9
+Wire Wire Line
+	7550 5500 7500 5500
+Connection ~ 7550 5500
+Wire Wire Line
+	8050 5500 8000 5500
+Connection ~ 8050 5500
+$Comp
+L MX_Alps_Hybrid:MX-NoLED MX45
+U 1 1 6141B38D
+P 8050 5350
+F 0 "MX45" H 8083 5573 60  0000 C CNN
+F 1 "MX-NoLED" H 8083 5499 20  0000 C CNN
+F 2 "MX_Only:MXOnly-2U-ReversedStabilizers-NoLED" H 7425 5325 60  0001 C CNN
+F 3 "" H 7425 5325 60  0001 C CNN
+	1    8050 5350
+	1    0    0    -1
+$EndComp
 $EndSCHEMATC
